File: rs232Isolator.kicad_pcb (KiCad board)
At the start: 2 copper layers, 40 x 30 mm, 31 parts, among them J1 DB9_Male, J2 DB9_Female, U1 MAX3232, U2 6N137, U3 6N137, U4 MAX3232

Commit message: throughole dsub connectors
Parts:
- J1: footprint Connector_Dsub:DSUB-9_Male_EdgeMount_P2.77mm -> Connector_Dsub:DSUB-9_Male_Horizontal_P2.77x2.84mm_EdgePinOffset9.90mm_Housed_MountingHolesOffset11.32mm
- J2: footprint Connector_Dsub:DSUB-9_Female_EdgeMount_P2.77mm -> Connector_Dsub:DSUB-9_Female_Horizontal_P2.77x2.84mm_EdgePinOffset9.90mm_Housed_MountingHolesOffset11.32mm
- R6, R7: value 1000 -> 1k
- moved J1 5.89 mm to (70.0, 79.5)
- moved J2 5.89 mm to (110.0, 79.5)
- moved G*** 2.00 mm to (78.0, 85.0)
Routing:
- net /5V2: track 25.0 -> 30.3 mm
- net /5V1: track 34.0 -> 38.9 mm
- net Net-(J2-Pad2): track 15.2 -> 17.2 mm
- net Net-(J2-Pad3): track 13.8 -> 15.8 mm
- net Net-(J1-Pad3): track 12.8 -> 14.8 mm
- net Net-(J1-Pad2): track 18.9 -> 20.9 mm
- net /Gnd2: track 52.3 -> 54.3 mm
- net /Gnd1: track 66.6 -> 68.6 mm
Other:
- board size 40 x 30 mm -> 48 x 30 mm
